File: Arduino_nano_v3.3/Arduino_nano_v3.3.kicad_pcb (KiCad board)
At the start: 2 copper layers, 17.8 x 43.2 mm, 34 parts, among them IC1 FT232RL, IC2 AMS117_3.3, IC3 Atmega_328p_AU, J1 Conn_01x15_Male, J2 Conn_01x15_Male, J3 USB_CON8, J4 ICSP_CONN_02X06, SW1 SW_Push, Y1 16MHz

Commit message: Layout design
Parts:
- removed TP1: D-, TestPoint:TestPoint_Pad_1.0x1.0mm
- removed TP2: D+, TestPoint:TestPoint_Pad_1.0x1.0mm
- RP1D1: moved to B.Cu
- moved RP1B1 44.0 mm to (124.0, 98.3), turned to 90 degrees
- moved C8 41.2 mm to (128.6, 84.7), turned to 90 degrees
- moved C7 39.4 mm to (126.8, 84.8), turned to 90 degrees
- moved D1 38.4 mm to (124.7, 87.8), turned to 270 degrees
- moved C9 29.5 mm to (133.9, 109.3), turned to 90 degrees
- moved C4 23.6 mm to (123.5, 104.7), turned to 270 degrees
- moved RP2C1 22.5 mm to (132.1, 82.3)
- moved C6 13.8 mm to (134.1, 95.5), turned to 90 degrees
- moved RP1A1 13.0 mm to (128.0, 105.9), turned to 90 degrees
- moved RP1D1 11.4 mm to (124.7, 83.7), turned to 90 degrees
- moved Y1 2.50 mm to (125.1, 89.0)
- moved IC3 0.16 mm to (129.1, 98.3)
Routing:
- net +5V: track 0.00 -> 85.6 mm, vias 0 -> 6
- net /RESET: track 0.00 -> 71.7 mm, vias 0 -> 3
- net /D13SCK: track 0.00 -> 47.3 mm, vias 0 -> 2
- net /D12MISO: track 0.00 -> 42.4 mm, vias 0 -> 2
- net GND: track 0.00 -> 38.1 mm, vias 0 -> 3
- net /D0RX: track 0.00 -> 38.0 mm, vias 0 -> 3
- net /VUSB: track 0.00 -> 37.8 mm, vias 0 -> 1
- net /D1TX: track 0.00 -> 33.5 mm, vias 0 -> 2
- net Net-(IC1-Pad22): track 0.00 -> 30.6 mm, vias 0 -> 1
- net Net-(IC1-Pad23): track 0.00 -> 27.0 mm, vias 0 -> 3
- net /A7: track 0.00 -> 20.9 mm, vias 0 -> 1
- net /A6: track 0.00 -> 18.5 mm, vias 0 -> 1
- net /D2: track 0.00 -> 15.1 mm, vias 0 -> 1
- net Net-(IC1-Pad15): track 0.00 -> 14.3 mm, vias 0 -> 1
- net VCC: track 0.00 -> 14.3 mm
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- added copper zone on B.Cu, net GND
- added copper zone on F.Cu, net GND

Commit message: Updated Layout design
Parts:
- RP1A1: moved to B.Cu
- moved C9 27.0 mm to (127.2, 83.1)
- moved RP1A1 19.2 mm to (132.8, 87.2), turned to 0 degrees
- moved C4 18.2 mm to (133.7, 89.6)
- moved C6 12.9 mm to (133.7, 108.5), turned to 270 degrees
- moved RP1B1 10.4 mm to (133.0, 93.0), turned to 180 degrees
- moved RP1D1 5.60 mm to (125.5, 78.1), turned to 270 degrees
- moved C8 3.99 mm to (127.9, 80.8), turned to 0 degrees
- moved C7 3.81 mm to (125.5, 81.2), turned to 270 degrees
- moved F1 3.19 mm to (131.8, 106.6)
- moved Y1 2.98 mm to (124.9, 91.9)
- moved IC1 2.46 mm to (128.8, 99.8), turned to 180 degrees
- moved IC2 2.33 mm to (128.2, 78.3), turned to 90 degrees
- moved C3 2.29 mm to (130.8, 78.0)
- moved C5 1.75 mm to (132.8, 78.7)
- moved C2 0.99 mm to (124.5, 107.9)
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Connections:
- J4 pad 4: /D1 -> /D1TX
Routing:
- net GND: track 38.1 -> 85.4 mm, vias 3 -> 11
- net /RESET: track 71.7 -> 43.4 mm
- net Net-(IC1-Pad22): track 30.6 -> 19.0 mm
- net Net-(IC1-Pad23): track 27.0 -> 18.7 mm, vias 3 -> 1
- net /RX: track 2.58 -> 10.7 mm, vias 1 -> 0
- net Net-(IC1-Pad15): track 14.3 -> 8.05 mm
- net /D0RX: track 38.0 -> 31.9 mm, vias 3 -> 1
- net Net-(IC1-Pad16): track 14.3 -> 8.95 mm
- net Net-(C4-Pad2): track 2.29 -> 7.53 mm
- net /D1TX: track 33.5 -> 38.1 mm, vias 2 -> 3
- net VCC: track 14.3 -> 9.77 mm
- net /A6: track 18.5 -> 21.9 mm
- net Net-(IC3-Pad8): track 8.24 -> 4.94 mm
- net Net-(IC3-Pad7): track 10.3 -> 7.04 mm
- net +3V3: track 14.1 -> 17.0 mm, vias 2 -> 0
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Other:
- rule via_min_size: 0.4 -> 0.2
