File: Arduino_nano_v3.3/Arduino_nano_v3.3.sch (KiCad schematic (older format))
At the start: 30 parts, among them IC1 FT232RL, IC2 AMS117_3.3, IC3 Atmega_328p_MUR, J1 Conn_01x15_Male, J2 Conn_01x15_Male, J3 USB_CON8, J4 ICSP_CONN_02X06, SW1 SW_Push, Y1 16MHz

Commit message: Changes in Shematics
Parts:
- added PWR? (x2): Green, symbol Device:LED
- added RP2B, RP2D: 1K, symbol Device:R
- IC2: footprint (none) -> Package_TO_SOT_SMD:SOT-23
- renumbered F to F1, L to L1, PWR to PWR1, RP1A to RP1A1, RP1B to RP1B1, RP1C to RP1C1, RP1D to RP1D1, RP2A to RP2A1, RP2C to RP2C1
Connections:
- net +5V: now also IC1.20 (VCC), PWR?.2 (A), PWR?.2 (A)
- net at IC1.22 (CBUS1): now also RP2D.1
- net at IC1.23 (CBUS0): now also RP2B.1
- new net: PWR?.1 (K), RP2B.2
- new net: PWR?.1 (K), RP2D.2

Commit message: Changes in Schematics
Parts:
- RX: renamed from PWR?; value Green -> Red
- gave numbers to parts that had none: 1
Changed lines of the file:
@@
 	9050 1850 7550 1850
 $Comp
-L Device:LED PWR?
+L Device:LED RX
 U 1 1 6088F451
 P 8575 975
-F 0 "PWR?" V 8614 1055 50  0000 L CNN
-F 1 "Green" V 8523 1055 50  0000 L CNN
+F 0 "RX" V 8614 1055 50  0000 L CNN
+F 1 "Red" V 8523 1055 50  0000 L CNN
 F 2 "" H 8575 975 50  0001 C CNN
 F 3 "~" H 8575 975 50  0001 C CNN
@@
 $EndComp
 $Comp
-L Device:LED PWR?
+L Device:LED TX
 U 1 1 60892440
 P 9050 975
-F 0 "PWR?" V 9089 1055 50  0000 L CNN
+F 0 "TX" V 9089 1055 50  0000 L CNN
 F 1 "Green" V 8998 1055 50  0000 L CNN
 F 2 "" H 9050 975 50  0001 C CNN

Commit message: Updated layout design
Parts:
- C1, C3, C4, C6, C7, C8, C9: footprint (none) -> Capacitor_SMD:C_0603_1608Metric
- C2, C5: footprint (none) -> Capacitor_SMD:C_1206_3216Metric
- D1: footprint Diode_THT:D_DO-201AD_P15.24mm_Horizontal -> Arduino_v3.3:SS1P3L_diode
- F1: footprint (none) -> Fuse:Fuse_0603_1608Metric
- IC3: value Atmega_328p_MUR -> Atmega_328p_AU
- J1, J2: footprint (none) -> Connector_PinHeader_2.54mm:PinHeader_1x15_P2.54mm_Vertical
- J3: footprint (none) -> Arduino_v3.3:Micro_usb_connector_4_THT_pads
- J4: footprint (none) -> Arduino_v3.3:ICSP_Arduino__connector
- L1, PWR1: footprint (none) -> LED_SMD:LED_0603_1608Metric
- RP1A1, RP1B1, RP1C1, RP1D1, RP2A1, RP2C1: footprint (none) -> Resistor_SMD:R_0603_1608Metric
- RP2B1: renamed from RP2B; footprint (none) -> Resistor_SMD:R_0603_1608Metric
- RP2D1: renamed from RP2D; footprint (none) -> Resistor_SMD:R_0603_1608Metric
- RX1: renamed from RX; footprint (none) -> LED_SMD:LED_0603_1608Metric
- SW1: footprint (none) -> Button_Switch_SMD:SW_SPST_B3U-1000P
- TP1, TP2: footprint (none) -> TestPoint:TestPoint_Pad_1.0x1.0mm
- TX1: renamed from TX; footprint (none) -> LED_SMD:LED_0603_1608Metric
- Y1: footprint (none) -> Arduino_v3.3:OSC_CSTCE16M0V53-R0
Connections:
- net 10 is gone; now on net D10: J1.13 (Pin_13)
- no-connect marks 0 -> 14
Changed lines of the file:
@@
 F 0 "D1" H 5700 7092 50  0000 C CNN
 F 1 "SS1P3L" H 5700 7001 50  0000 C CNN
-F 2 "Diode_THT:D_DO-201AD_P15.24mm_Horizontal" H 5700 6700 50  0001 C CNN
+F 2 "Arduino_v3.3:SS1P3L_diode" H 5700 6700 50  0001 C CNN
 F 3 "http://www.vishay.com/docs/88516/1n5400.pdf" H 5700 6875 50  0001 C CNN
 	1    5700 6875
@@
 F 0 "J3" H 9975 3215 50  0000 C CNN
 F 1 "USB_CON8" H 9975 3124 50  0000 C CNN
-F 2 "" H 10325 3400 50  0001 C CNN
+F 2 "Arduino_v3.3:Micro_usb_connector_4_THT_pads" H 10325 3400 50  0001 C CNN
 F 3 "" H 10325 3400 50  0001 C CNN
 	1    9875 2800
@@
 P 4600 3675
 F 0 "IC3" H 4950 4040 50  0000 C CNN
-F 1 "Atmega_328p_MUR" H 4950 3949 50  0000 C CNN
+F 1 "Atmega_328p_AU" H 4950 3949 50  0000 C CNN
 F 2 "Package_QFP:TQFP-32_7x7mm_P0.8mm" H 4700 4525 50  0001 C CNN
 F 3 "" H 4700 4525 50  0001 C CNN
@@
 F 0 "J1" H 2150 2975 50  0000 R CNN
 F 1 "Conn_01x15_Male" H 2250 2825 50  0000 R CNN
-F 2 "" H 1925 2000 50  0001 C CNN
+F 2 "Connector_PinHeader_2.54mm:PinHeader_1x15_P2.54mm_Vertical" H 1925 2000 50  0001 C CNN
 F 3 "~" H 1925 2000 50  0001 C CNN
 	1    1925 2000
@@
 F 0 "J2" H 3058 2881 50  0000 C CNN
 F 1 "Conn_01x15_Male" H 3058 2790 50  0000 C CNN
-F 2 "" H 2950 2000 50  0001 C CNN
+F 2 "Connector_PinHeader_2.54mm:PinHeader_1x15_P2.54mm_Vertical" H 2950 2000 50  0001 C CNN
 F 3 "~" H 2950 2000 50  0001 C CNN
 	1    2950 2000
@@
 D9
 Text Label 1325 2500 0    50   ~ 0
-10
+D10
 Text Label 1325 2600 0    50   ~ 0
 D11MOSI
@@
 F 0 "SW1" H 1175 4260 50  0000 C CNN
 F 1 "SW_Push" H 1175 4169 50  0000 C CNN
-F 2 "" H 1175 4175 50  0001 C CNN
+F 2 "Button_Switch_SMD:SW_SPST_B3U-1000P" H 1175 4175 50  0001 C CNN
 F 3 "~" H 1175 4175 50  0001 C CNN
 	1    1175 3975
@@
 F 0 "RP1D1" H 1795 3621 50  0000 L CNN
 F 1 "1K" H 1795 3530 50  0000 L CNN
-F 2 "" V 1655 3575 50  0001 C CNN
+F 2 "Resistor_SMD:R_0603_1608Metric" V 1655 3575 50  0001 C CNN
 F 3 "~" H 1725 3575 50  0001 C CNN
 	1    1725 3575
@@
 F 0 "Y1" V 3175 3750 50  0000 L CNN
 F 1 "16MHz" V 3275 3475 50  0000 L CNN
-F 2 "" H 3375 3925 50  0001 C CNN
+F 2 "Arduino_v3.3:OSC_CSTCE16M0V53-R0" H 3375 3925 50  0001 C CNN
 F 3 "~" H 3375 3925 50  0001 C CNN
 	1    3400 3925
@@
 F 0 "C1" H 1615 4696 50  0000 L CNN
 F 1 "100nF" H 1615 4605 50  0000 L CNN
-F 2 "" H 1538 4500 50  0001 C CNN
+F 2 "Capacitor_SMD:C_0603_1608Metric" H 1538 4500 50  0001 C CNN
 F 3 "~" H 1500 4650 50  0001 C CNN
 	1    1500 4650
@@
 F 0 "C5" H 2768 5496 50  0000 L CNN
 F 1 "4.7uF_16V" H 2675 5350 50  0000 L CNN
-F 2 "" H 2688 5300 50  0001 C CNN
+F 2 "Capacitor_SMD:C_1206_3216Metric" H 2688 5300 50  0001 C CNN
 F 3 "~" H 2650 5450 50  0001 C CNN
 	1    2650 5450
@@
 F 0 "C7" H 2090 5496 50  0000 L CNN
 F 1 "1uF" H 2090 5405 50  0000 L CNN
-F 2 "" H 2013 5300 50  0001 C CNN
+F 2 "Capacitor_SMD:C_0603_1608Metric" H 2013 5300 50  0001 C CNN
 F 3 "~" H 1975 5450 50  0001 C CNN
 	1    1975 5450
@@
 F 0 "C3" H 3290 5496 50  0000 L CNN
 F 1 "1uF" H 3290 5405 50  0000 L CNN
-F 2 "" H 3213 5300 50  0001 C CNN
+F 2 "Capacitor_SMD:C_0603_1608Metric" H 3213 5300 50  0001 C CNN
 F 3 "~" H 3175 5450 50  0001 C CNN
 	1    3175 5450
@@
 F 0 "RP1B1" V 6693 5625 50  0000 C CNN
 F 1 "1K" V 6784 5625 50  0000 C CNN
-F 2 "" V 6830 5625 50  0001 C CNN
+F 2 "Resistor_SMD:R_0603_1608Metric" V 6830 5625 50  0001 C CNN
 F 3 "~" H 6900 5625 50  0001 C CNN
 	1    6900 5625
@@
 F 0 "RP1A1" V 6693 6000 50  0000 C CNN
 F 1 "1K" V 6784 6000 50  0000 C CNN
-F 2 "" V 6830 6000 50  0001 C CNN
+F 2 "Resistor_SMD:R_0603_1608Metric" V 6830 6000 50  0001 C CNN
 F 3 "~" H 6900 6000 50  0001 C CNN
 	1    6900 6000
@@
 F 0 "RP2A1" H 6930 4079 50  0000 R CNN
 F 1 "1K" H 6930 4170 50  0000 R CNN
-F 2 "" V 6930 4125 50  0001 C CNN
+F 2 "Resistor_SMD:R_0603_1608Metric" V 6930 4125 50  0001 C CNN
 F 3 "~" H 7000 4125 50  0001 C CNN
 	1    7000 4125
@@
 F 0 "L1" V 7039 4755 50  0000 L CNN
 F 1 "YELLOW" V 6948 4755 50  0000 L CNN
-F 2 "" H 7000 4675 50  0001 C CNN
+F 2 "LED_SMD:LED_0603_1608Metric" H 7000 4675 50  0001 C CNN
 F 3 "~" H 7000 4675 50  0001 C CNN
 	1    7000 4675
@@
 F 0 "C8" H 3690 7221 50  0000 L CNN
 F 1 "1uF" H 3690 7130 50  0000 L CNN
-F 2 "" H 3613 7025 50  0001 C CNN
+F 2 "Capacitor_SMD:C_0603_1608Metric" H 3613 7025 50  0001 C CNN
 F 3 "~" H 3575 7175 50  0001 C CNN
 	1    3575 7175
@@
 F 0 "RP1C1" V 3868 6925 50  0000 C CNN
 F 1 "1K" V 3959 6925 50  0000 C CNN
-F 2 "" V 4005 6925 50  0001 C CNN
+F 2 "Resistor_SMD:R_0603_1608Metric" V 4005 6925 50  0001 C CNN
 F 3 "~" H 4075 6925 50  0001 C CNN
 	1    4075 6925
@@
 F 0 "PWR1" V 4614 7230 50  0000 L CNN
 F 1 "Green" V 4523 7230 50  0000 L CNN
-F 2 "" H 4575 7150 50  0001 C CNN
+F 2 "LED_SMD:LED_0603_1608Metric" H 4575 7150 50  0001 C CNN
 F 3 "~" H 4575 7150 50  0001 C CNN
 	1    4575 7150
@@
 F 0 "J4" H 8575 6440 50  0000 C CNN
 F 1 "ICSP_CONN_02X06" H 8575 6349 50  0000 C CNN
-F 2 "" H 8575 5975 50  0001 C CNN
+F 2 "Arduino_v3.3:ICSP_Arduino__connector" H 8575 5975 50  0001 C CNN
 F 3 "" H 8575 5975 50  0001 C CNN
 	1    8575 5975
@@
 Wire Wire Line
 	8175 5975 7725 5975
-Wire Wire Line
-	8975 5875 9525 5875
 Text Label 7725 5775 0    50   ~ 0
 D12MISO
@@
 F 0 "C2" H 10218 5196 50  0000 L CNN
 F 1 "4.7uF_16V" H 10125 5050 50  0000 L CNN
-F 2 "" H 10138 5000 50  0001 C CNN
+F 2 "Capacitor_SMD:C_1206_3216Metric" H 10138 5000 50  0001 C CNN
 F 3 "~" H 10100 5150 50  0001 C CNN
 	1    10100 5150
@@
 F 0 "C9" H 10915 5171 50  0000 L CNN
 F 1 "100nF" H 10915 5080 50  0000 L CNN
-F 2 "" H 10838 4975 50  0001 C CNN
+F 2 "Capacitor_SMD:C_0603_1608Metric" H 10838 4975 50  0001 C CNN
 F 3 "~" H 10800 5125 50  0001 C CNN
 	1    10800 5125
@@
 F 0 "RP2C1" V 8057 4400 50  0000 C CNN
 F 1 "1K" V 7966 4400 50  0000 C CNN
-F 2 "" V 7780 4400 50  0001 C CNN
+F 2 "Resistor_SMD:R_0603_1608Metric" V 7780 4400 50  0001 C CNN
 F 3 "~" H 7850 4400 50  0001 C CNN
 	1    7850 4400
@@
 F 0 "C4" V 5527 1350 50  0000 C CNN
 F 1 "100nF" V 5436 1350 50  0000 C CNN
-F 2 "" H 5313 1200 50  0001 C CNN
+F 2 "Capacitor_SMD:C_0603_1608Metric" H 5313 1200 50  0001 C CNN
 F 3 "~" H 5275 1350 50  0001 C CNN
 	1    5275 1350
@@
 F 0 "C6" H 8165 3196 50  0000 L CNN
 F 1 "100nF" H 8165 3105 50  0000 L CNN
-F 2 "" H 8088 3000 50  0001 C CNN
+F 2 "Capacitor_SMD:C_0603_1608Metric" H 8088 3000 50  0001 C CNN
 F 3 "~" H 8050 3150 50  0001 C CNN
 	1    8050 3150
@@
 F 0 "F1" V 8500 2650 50  0000 C CNN
 F 1 "Polyfuse" V 8591 2650 50  0000 C CNN
-F 2 "" H 8775 2450 50  0001 L CNN
+F 2 "Fuse:Fuse_0603_1608Metric" H 8775 2450 50  0001 L CNN
 F 3 "~" H 8725 2650 50  0001 C CNN
 	1    8725 2650
@@
 F 0 "TP2" H 8392 3501 50  0000 R CNN
 F 1 "D+" H 8392 3592 50  0000 R CNN
-F 2 "" H 8650 3475 50  0001 C CNN
+F 2 "TestPoint:TestPoint_Pad_1.0x1.0mm" H 8650 3475 50  0001 C CNN
 F 3 "~" H 8650 3475 50  0001 C CNN
 	1    8450 3475
@@
 F 0 "TP1" H 8717 3176 50  0000 R CNN
 F 1 "D-" H 8717 3267 50  0000 R CNN
-F 2 "" H 8975 3150 50  0001 C CNN
+F 2 "TestPoint:TestPoint_Pad_1.0x1.0mm" H 8975 3150 50  0001 C CNN
 F 3 "~" H 8975 3150 50  0001 C CNN
 	1    8775 3150
@@
 	10600 2950 10600 3275
 $Comp
-L Device:R RP2B
+L Device:R RP2B1
 U 1 1 60878FA5
 P 8575 1375
-F 0 "RP2B" H 8505 1329 50  0000 R CNN
+F 0 "RP2B1" H 8505 1329 50  0000 R CNN
 F 1 "1K" H 8505 1420 50  0000 R CNN
-F 2 "" V 8505 1375 50  0001 C CNN
+F 2 "Resistor_SMD:R_0603_1608Metric" V 8505 1375 50  0001 C CNN
 F 3 "~" H 8575 1375 50  0001 C CNN
 	1    8575 1375
@@
 $EndComp
 $Comp
-L Device:R RP2D
+L Device:R RP2D1
 U 1 1 6087ADA2
 P 9050 1400
-F 0 "RP2D" H 8980 1354 50  0000 R CNN
+F 0 "RP2D1" H 8980 1354 50  0000 R CNN
 F 1 "1K" H 8980 1445 50  0000 R CNN
-F 2 "" V 8980 1400 50  0001 C CNN
+F 2 "Resistor_SMD:R_0603_1608Metric" V 8980 1400 50  0001 C CNN
 F 3 "~" H 9050 1400 50  0001 C CNN
 	1    9050 1400
@@
 	9050 1850 7550 1850
 $Comp
-L Device:LED RX
+L Device:LED RX1
 U 1 1 6088F451
 P 8575 975
-F 0 "RX" V 8614 1055 50  0000 L CNN
+F 0 "RX1" V 8614 1055 50  0000 L CNN
 F 1 "Red" V 8523 1055 50  0000 L CNN
-F 2 "" H 8575 975 50  0001 C CNN
+F 2 "LED_SMD:LED_0603_1608Metric" H 8575 975 50  0001 C CNN
 F 3 "~" H 8575 975 50  0001 C CNN
 	1    8575 975
@@
 $EndComp
 $Comp
-L Device:LED TX
+L Device:LED TX1
 U 1 1 60892440
 P 9050 975
-F 0 "TX" V 9089 1055 50  0000 L CNN
+F 0 "TX1" V 9089 1055 50  0000 L CNN
 F 1 "Green" V 8998 1055 50  0000 L CNN
-F 2 "" H 9050 975 50  0001 C CNN
+F 2 "LED_SMD:LED_0603_1608Metric" H 9050 975 50  0001 C CNN
 F 3 "~" H 9050 975 50  0001 C CNN
 	1    9050 975
@@
 $EndComp
 $Comp
-L power:+5V #PWR?
+L power:+5V #PWR01
 U 1 1 60892C04
 P 8050 725
-F 0 "#PWR?" H 8050 575 50  0001 C CNN
+F 0 "#PWR01" H 8050 575 50  0001 C CNN
 F 1 "+5V" H 8065 898 50  0000 C CNN
 F 2 "" H 8050 725 50  0001 C CNN
@@
 $EndComp
 $Comp
-L power:+5V #PWR?
+L power:+5V #PWR02
 U 1 1 608933D0
 P 8575 725
-F 0 "#PWR?" H 8575 575 50  0001 C CNN
+F 0 "#PWR02" H 8575 575 50  0001 C CNN
 F 1 "+5V" H 8590 898 50  0000 C CNN
 F 2 "" H 8575 725 50  0001 C CNN
@@
 $EndComp
 $Comp
-L power:+5V #PWR?
+L power:+5V #PWR03
 U 1 1 6089376A
 P 9050 725
-F 0 "#PWR?" H 9050 575 50  0001 C CNN
+F 0 "#PWR03" H 9050 575 50  0001 C CNN
 F 1 "+5V" H 9065 898 50  0000 C CNN
 F 2 "" H 9050 725 50  0001 C CNN
@@
 Wire Wire Line
 	8050 1250 8050 725
+NoConn ~ 9225 2950
+NoConn ~ 7550 1450
+NoConn ~ 7550 1550
+NoConn ~ 7550 1650
+NoConn ~ 7550 1950
+NoConn ~ 7550 2050
+NoConn ~ 7550 2150
+NoConn ~ 7550 2350
+NoConn ~ 5950 2150
+NoConn ~ 5950 2050
+NoConn ~ 5950 1950
+NoConn ~ 5950 1850
+NoConn ~ 5950 1750
+NoConn ~ 5950 1450
+Wire Wire Line
+	8975 5875 9525 5875
 $EndSCHEMATC

Commit message: Updated Layout design
Connections:
- net D1 is gone; now on net D1TX: J4.4
Changed lines of the file:
@@
 RESET
 Text Label 9525 5875 2    50   ~ 0
-D1
+D1TX
 $Comp
 L power:+5V #PWR0120
