File: Arduino_UNO_rev3/Arduino_UNO_rev3.sch (KiCad schematic (older format))
At the start: 61 parts, among them J1 USB_B_Micro, J2 ICSP_CONN_02X06, J3 Conn_02x02_Odd_Even, J4 Conn_01x08_Male, J5 ICSP_CONN_02X06, J6 Conn_01x10_Male, J7 Conn_01x06_Male, J8 Conn_01x08_Male, Q1 FDN340P, SW1 SW_MEC_5E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

Commit message: Adding footprints and layout
Parts:
- C1, C10, C11, C12, C13, C2, C5, C6, C7, C8, C9: footprint (none) -> Capacitor_SMD:C_0603_1608Metric
- C3, C4: footprint (none) -> Capacitor_THT:CP_Radial_D4.0mm_P1.50mm
- D1, D3, D5, D6: footprint (none) -> LED_SMD:LED_0603_1608Metric
- D2, D4, D7, D8, D9: footprint (none) -> Diode_SMD:D_0603_1608Metric
- F1: footprint (none) -> Fuse:Fuse_0603_1608Metric
- GD1, U5, U5B1: footprint (none) -> Arduino_UNO_rev3:MSOP08
- J1: footprint (none) -> Arduino_UNO_rev3:PN61729
- J2, J5: footprint (none) -> Arduino_v3.3:ICSP_Arduino__connector
- J3: footprint (none) -> Arduino_UNO_rev3:2X02
- J4, J8: footprint (none) -> Arduino_UNO_rev3:1X08
- J6: footprint (none) -> Arduino_UNO_rev3:1X10
- J7: footprint (none) -> Arduino_UNO_rev3:1X06
- L1, L2: footprint (none) -> Arduino_UNO_rev3:0805
- R1, R10, R11, R12, R13, R14, R15, R16, R2, R3, R4, R5, R6, R7, R8, R9: footprint (none) -> Resistor_SMD:R_0603_1608Metric
- SW1: footprint (none) -> Arduino_UNO_rev3:TS42
- U1: footprint (none) -> Arduino_UNO_rev3:SOT223
- U2: footprint (none) -> Arduino_UNO_rev3:POWERSUPPLY_DC-21MM
- U3: footprint Package_TO_SOT_SMD:SOT-23-5 -> Arduino_UNO_rev3:SOT23-DBV
- Y1: footprint (none) -> Arduino_UNO_rev3:QS
- Y2: footprint (none) -> Arduino_UNO_rev3:RESONATOR

Commit message: Updated schematics and footprint layout
Parts:
- removed GD1: GDT_2pin, Arduino_UNO_rev3:MSOP08, symbol Device:GDT_2pin
- removed R1, R10, R12, R13, R14, R15, R16, R2, R3, R4, R5, R6, R8, R9: R, Resistor_SMD:R_0603_1608Metric, symbol Device:R
- removed U5, U5B1: LMV358, Arduino_UNO_rev3:MSOP08, symbol Amplifier_Operational:LMV358
- added U10: RN3, Arduino_UNO_rev3:CAY16, symbol Memory_EEPROM:AT24CS64-MAHM
- added U5: RN1, Arduino_UNO_rev3:CAY16, symbol Memory_EEPROM:AT24CS64-MAHM
- added U7: RN2, Arduino_UNO_rev3:CAY16, symbol Memory_EEPROM:AT24CS64-MAHM
- added U8: LMV358IDGKR, Arduino_UNO_rev3:MSOP08, symbol Amplifier_Audio:LM386
- added U9: RN4, Arduino_UNO_rev3:CAY16, symbol Memory_EEPROM:AT24CS64-MAHM
- C1, C10, C11, C12, C13, C2, C5, C6, C7, C8, C9: footprint Capacitor_SMD:C_0603_1608Metric -> Arduino_UNO_rev3:C0603-ROUND
- C3, C4: footprint Capacitor_THT:CP_Radial_D4.0mm_P1.50mm -> Arduino_UNO_rev3:PANASONIC_D
- D1, D5, D6: footprint LED_SMD:LED_0603_1608Metric -> Arduino_UNO_rev3:CHIP-LED0805
- D2: footprint Diode_SMD:D_0603_1608Metric -> Arduino_UNO_rev3:SMB
- D4, D7: footprint Diode_SMD:D_0603_1608Metric -> Arduino_UNO_rev3:MINIMELF
- D8, D9: footprint Diode_SMD:D_0603_1608Metric -> Arduino_UNO_rev3:CT_CN0603
- F1: footprint Fuse:Fuse_0603_1608Metric -> Arduino_UNO_rev3:L1812
- J2, J5: footprint Arduino_v3.3:ICSP_Arduino__connector -> Arduino_UNO_rev3:ICSP_Arduino__connector_UNO
- R1: renamed from R11; footprint Resistor_SMD:R_0603_1608Metric -> Arduino_UNO_rev3:R0603-ROUND
- R2: renamed from R7; footprint Resistor_SMD:R_0603_1608Metric -> Arduino_UNO_rev3:R0603-ROUND
Connections:
- net +3V3: now also U8.2 (-)
- net +5V: now also C1.1, D7.1 (K), J2.2, U5.3 (A2), U5.5 (SDA), U7.2 (A1), U7.3 (A2), U8.8 (GAIN), U9.3 (A2), U9.4 (GND); no longer C1.2
- net CMP: now also U5.1 (A0), U5.2 (A1), U8.3 (+)
- net D+: now also U10.5 (SDA)
- net D-: now also U10.8 (VCC)
- net GATE_CMD: now also U8.1 (GAIN)
- net GND: now also C1.2, U5.7 (WP), U7.5 (SDA), U8.4 (GND); no longer C1.1
- net IO0: now also U9.2 (A1)
- net IO1: now also U9.1 (A0)
- net L13: now also U7.8 (VCC), U8.6 (V+), U8.7 (BYPASS)
- net M8RXD: now also U9.7 (WP)
- net M8TXD: now also U9.8 (VCC)
- net RD+: now also U10.4 (GND)
- net RD-: now also U10.1 (A0)
- net RESET: now also U5.4 (GND)
- net RESET2: now also U5.6 (SCL)
- net SCK: now also U8.5
- net VIN: now also U5.8 (VCC)
- net RN2P4: now reaches C9.1, U4.13 (~HWB~/PD7)
- net RN2P4: now also U7.4 (GND)
- net RN2P6: now reaches D5.2 (A)
- net RN2P6: now also U7.6 (SCL)
- net RN2P7: now reaches D6.2 (A)
- net RN2P7: now also U7.7 (WP)
- net at D1.2 (A): now also U7.1 (A0)
- net at D3.2 (A): now also U9.5 (SDA), U9.6 (SCL)
- no-connect marks 11 -> 15
Other:
- moved on the sheet: C1, D1, D3
