File: Arduino_UNO_rev3/Arduino_UNO_rev3.kicad_pcb (KiCad board)
At the start: 2 copper layers, 68.6 x 53.4 mm, 49 parts, among them J1 USB_B_Micro, J2 ICSP_CONN_02X06, J3 Conn_02x02_Odd_Even, J4 Conn_01x08_Male, J5 ICSP_CONN_02X06, J6 Conn_01x10_Male, J7 Conn_01x06_Male, J8 Conn_01x08_Male, Q1 FDN340P, SW1 SW_MEC_5E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

Commit message: Copplete routings and layout desig
Parts:
- moved J3 0.83 mm to (160.2, 63.3)
Routing:
- net +5V: track 0.00 -> 200.7 mm, vias 0 -> 5
- net /RESET: track 0.00 -> 151.4 mm, vias 0 -> 3
- net /SCK: track 0.00 -> 127.5 mm, vias 0 -> 2
- net /AD5SCL: track 0.00 -> 114.0 mm, vias 0 -> 1
- net /AD4SDA: track 0.00 -> 112.5 mm
- net /MOSI: track 0.00 -> 102.8 mm, vias 0 -> 1
- net GND: track 0.00 -> 93.8 mm, vias 0 -> 12
- net /MISO: track 0.00 -> 92.2 mm, vias 0 -> 1
- net /AREF: track 0.00 -> 83.5 mm, vias 0 -> 1
- net /VIN: track 0.00 -> 64.9 mm, vias 0 -> 3
- net /IO9: track 0.00 -> 58.8 mm, vias 0 -> 1
- net /SS: track 0.00 -> 56.4 mm, vias 0 -> 1
- net /IO8: track 0.00 -> 50.0 mm
- net /L13: track 0.00 -> 47.8 mm, vias 0 -> 2
- net /IO7: track 0.00 -> 46.2 mm
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- added copper zone on F.Cu, net +5V
- added copper zone on B.Cu, net GND
- added copper zone on F.Cu, net GND
